File: MARS-Rover-Pico-Adapter/MARS-Rover-Pico-Adapter.kicad_pcb (KiCad board)
At the start: 2 copper layers, 63 x 64 mm, 7 parts, among them J3 Conn_02x20_Odd_Even, U1 Pico

Commit message: Update adapter board
Parts:
- removed J1: ~, rover_custom_footprints:PS2_Remote board
- added J2: Conn_01x04_Pin, Connector_PinHeader_2.54mm:PinHeader_1x04_P2.54mm_Vertical, F.Cu at (154.0, 66.8)
- added J4: Conn_01x06_Pin, Connector_PinHeader_2.54mm:PinHeader_1x06_P2.54mm_Vertical, F.Cu at (75.0, 90.3)
- added JP1: SolderJumper_3_Bridged12, Jumper:SolderJumper-3_P1.3mm_Bridged12_RoundedPad1.0x1.5mm, F.Cu at (83.3, 87.8)
- added REF**: MountingHole_2.5mm, MountingHole:MountingHole_2.5mm, F.Cu at (89.0, 109.5)
- added REF**: MountingHole_2.5mm, MountingHole:MountingHole_2.5mm, F.Cu at (89.0, 58.5)
- added REF**: MountingHole_2.5mm, MountingHole:MountingHole_2.5mm, F.Cu at (74.0, 98.0)
- added REF**: MountingHole_2.5mm, MountingHole:MountingHole_2.5mm, F.Cu at (74.0, 70.0)
- added SW1: SW_Push, Button_Switch_THT:SW_PUSH_6mm, F.Cu at (156.4, 105.0)
- added SW2: SW_Push, Button_Switch_THT:SW_PUSH_6mm, F.Cu at (162.9, 63.0)
Connections:
- net Ultrasonic renamed Ultrasonic1
- J3 pad 10: unconnected-(J3-Pin_10-Pad10) -> GND
- J3 pad 13: unconnected-(J3-Pin_13-Pad13) -> GND
- J3 pad 17: unconnected-(J3-Pin_17-Pad17) -> Ultrasonic2
- J3 pad 19: unconnected-(J3-Pin_19-Pad19) -> GND
- J3 pad 21: unconnected-(J3-Pin_21-Pad21) -> Ultrasonic3
- J3 pad 26: unconnected-(J3-Pin_26-Pad26) -> GND
- J3 pad 29: unconnected-(J3-Pin_29-Pad29) -> GND
- J3 pad 30: unconnected-(J3-Pin_30-Pad30) -> Ultrasonic4
- J3 pad 33: unconnected-(J3-Pin_33-Pad33) -> GND
- J3 pad 40: unconnected-(J3-Pin_40-Pad40) -> GND
- U1 pad 21: Remote_Data_Out -> Remote_Cmd
- U1 pad 25: Remote_Data_In -> Remote_Data
- U1 pad 26: Remote_ACK -> BUTTON_L
- U1 pad 27: unconnected-(U1-GPIO21-Pad27)_1 -> BUTTON_R
- U1 pad 31: unconnected-(U1-GPIO26_ADC0-Pad31) -> SCREEN_SDA
- U1 pad 32: unconnected-(U1-GPIO27_ADC1-Pad32)_1 -> SCREEN_SCL
- U1 pad 42: unconnected-(U1-GND-Pad42) -> GND
- U1 pad 6: unconnected-(U1-GPIO4-Pad6)_1 -> Ultrasonic2
- U1 pad 7: unconnected-(U1-GPIO5-Pad7)_1 -> Ultrasonic3
- U1 pad 9: unconnected-(U1-GPIO6-Pad9) -> Ultrasonic4
Routing:
- net +3V3: track 18.8 -> 111.8 mm
- net Remote_Cmd: track 0.00 -> 67.3 mm
- net BUTTON_R: track 0.00 -> 65.2 mm
- net Remote_Data: track 0.00 -> 53.1 mm
- net SCREEN_SDA: track 0.00 -> 49.5 mm
- net BUTTON_L: track 0.00 -> 47.4 mm
- net SCREEN_SCL: track 0.00 -> 46.9 mm
- net +5V: track 32.2 -> 66.3 mm
- net Remote_CS: track 29.7 -> 62.6 mm
- net Remote_ACK: track 31.3 -> 0.00 mm
- net Remote_CLK: track 28.8 -> 50.8 mm
- net Ultrasonic4: track 0.00 -> 19.4 mm
- net Ultrasonic3: track 0.00 -> 16.5 mm
- net Remote_Data_Out: track 16.4 -> 0.00 mm
- net Ultrasonic2: track 0.00 -> 13.6 mm
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Other:
- board size 63 x 64 mm -> 93.5 x 64 mm
- board text added: "+3V3"
- board text added: "+5V"
- board text added: "ATT"
- board text added: "CLK"
- board text added: "CMD"
- board text added: "DAT"
- board text added: "GND"
- board text added: "M.A.R.S. rover RPi Pico Adapter v2.0"
- board text added: "SCL"
- board text added: "SDA"
- board text added: "VCC->"
- board text removed: "M.A.R.S. rover RPi Pico Adapter v1.0"
- board text removed: "PS2 Remote Controller"
