File: MARS-Rover-Pico-Adapter/MARS-Rover-Pico-Adapter.kicad_sch (KiCad schematic)
At the start: 3 parts, among them J3 Conn_02x20_Odd_Even, U1 Pico

Commit message: Update adapter board
Parts:
- removed J1: ~, rover_custom_footprints:PS2_Remote board, symbol symbol_library:ps2_controller
- added J2: Conn_01x04_Pin, Connector_PinHeader_2.54mm:PinHeader_1x04_P2.54mm_Vertical, symbol Connector:Conn_01x04_Pin
- added J4: Conn_01x06_Pin, Connector_PinHeader_2.54mm:PinHeader_1x06_P2.54mm_Vertical, symbol Connector:Conn_01x06_Pin
- added JP1: SolderJumper_3_Bridged12, Jumper:SolderJumper-3_P1.3mm_Bridged12_RoundedPad1.0x1.5mm, symbol Jumper:SolderJumper_3_Bridged12
- added SW1, SW2: SW_Push, Button_Switch_THT:SW_PUSH_6mm, symbol Switch:SW_Push
Connections:
- net +3V3: now also J2.2 (Pin_2), JP1.1 (A)
- net +5V: now also JP1.3 (B)
- net GND: now also J3.10 (Pin_10), J3.13 (Pin_13), J3.19 (Pin_19), J3.26 (Pin_26), J3.29 (Pin_29), J3.33 (Pin_33), J3.40 (Pin_40), U1.42 (GND), J2.1 (Pin_1), J4.1 (Pin_1), SW1.2, SW2.2
- net Remote_CLK: now also J4.3 (Pin_3)
- net Remote_CS: now also J4.4 (Pin_4)
- net Ultrasonic2: now reaches J3.17 (Pin_17)
- net Ultrasonic2: now also U1.6 (GPIO4)
- net Ultrasonic3: now reaches J3.21 (Pin_21)
- net Ultrasonic3: now also U1.7 (GPIO5)
- net Ultrasonic4: now reaches J3.30 (Pin_30)
- net Ultrasonic4: now also U1.9 (GPIO6)
- net BUTTON_R: now reaches U1.27 (GPIO21)
- net BUTTON_R: now also SW2.1
- net SCREEN_SDA: now reaches U1.31 (GPIO26_ADC0)
- net SCREEN_SDA: now also J2.4 (Pin_4)
- net SCREEN_SCL: now reaches U1.32 (GPIO27_ADC1)
- net SCREEN_SCL: now also J2.3 (Pin_3)
- net Remote_ACK renamed BUTTON_L
- net BUTTON_L: now also SW1.1
- net Remote_Data_In renamed Remote_Data
- net Remote_Data: now also J4.6 (Pin_6)
- net Remote_Data_Out renamed Remote_Cmd
- net Remote_Cmd: now also J4.5 (Pin_5)
- net Ultrasonic renamed Ultrasonic1
- new net Remote_VCC: J4.2 (Pin_2), JP1.2 (C)
- no-connect marks 48 -> 33
Other:
- note added: "#05"
- note added: "#18"
- note added: "#23"
- note added: "#24"
- note added: "#25"
- note added: "I2C1"
